File: untitled.sch (EAGLE design)
At the start: 109 parts, among them IC1 STM32F103ZET6, IC2 PL2303TA, IC3 24C16BSN, IC4 LM393D, Q1 IRF510, Q2 IRF510, Q3 IRF510, Q4 IRF510, Q5 IRF510, Q6 IRF510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

Commit message: Add files via upload
Connections:
- net N$62: now also IC1.PB8; no longer IC1.PB9
- net N$72: now also IC1.PB9; no longer IC1.PB8
Changed lines of the file:
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@@
 <net name="N$62" class="0">
 <segment>
-<pinref part="IC1" gate="G$1" pin="PB9"/>
-<wire x1="80.01" y1="53.34" x2="80.01" y2="66.04" width="0.1524" layer="91"/>
 <pinref part="U2" gate="G$1" pin="!ENABLE"/>
 <wire x1="-58.42" y1="60.96" x2="-40.64" y2="60.96" width="0.1524" layer="91"/>
 <wire x1="-40.64" y1="60.96" x2="-33.02" y2="60.96" width="0.1524" layer="91"/>
 <wire x1="-33.02" y1="60.96" x2="-33.02" y2="66.04" width="0.1524" layer="91"/>
-<wire x1="-33.02" y1="66.04" x2="80.01" y2="66.04" width="0.1524" layer="91"/>
+<wire x1="-33.02" y1="66.04" x2="79.756" y2="66.04" width="0.1524" layer="91"/>
 <pinref part="R48" gate="G$1" pin="1"/>
+<wire x1="79.756" y1="66.04" x2="80.01" y2="66.04" width="0.1524" layer="91"/>
 <wire x1="-40.64" y1="83.82" x2="-40.64" y2="60.96" width="0.1524" layer="91"/>
 <junction x="-40.64" y="60.96"/>
+<pinref part="IC1" gate="G$1" pin="PB8"/>
+<wire x1="82.55" y1="53.34" x2="82.55" y2="66.04" width="0.1524" layer="91"/>
+<wire x1="82.55" y1="66.04" x2="80.01" y2="66.04" width="0.1524" layer="91"/>
 </segment>
 </net>
@@
 <wire x1="-58.42" y1="20.32" x2="-30.48" y2="20.32" width="0.1524" layer="91"/>
 <wire x1="-30.48" y1="20.32" x2="-30.48" y2="63.5" width="0.1524" layer="91"/>
-<wire x1="-30.48" y1="63.5" x2="82.55" y2="63.5" width="0.1524" layer="91"/>
-<pinref part="IC1" gate="G$1" pin="PB8"/>
-<wire x1="82.55" y1="53.34" x2="82.55" y2="63.5" width="0.1524" layer="91"/>
+<wire x1="-30.48" y1="63.5" x2="76.2" y2="63.5" width="0.1524" layer="91"/>
+<pinref part="IC1" gate="G$1" pin="PB9"/>
+<wire x1="76.2" y1="63.5" x2="76.454" y2="63.5" width="0.1524" layer="91"/>
+<wire x1="80.01" y1="53.34" x2="80.01" y2="63.5" width="0.1524" layer="91"/>
+<wire x1="80.01" y1="63.5" x2="76.454" y2="63.5" width="0.1524" layer="91"/>
 </segment>
 </net>
